File: display.kicad_sch (KiCad schematic)
At the start: 20 parts, among them U201 QS6K1FRATR, U202 LTP-3784E, U203 PCA9685PW

Commit message: finish routing(?)
Connections:
- net at R206.1: now also U203.9 (LED3); no longer U202.5 (K)
- net at R206.2: now also U202.5 (K); no longer U203.9 (LED3)
- net at R203.1: now also U203.6 (LED0); no longer U202.1 (E)
- net at R203.2: now also U202.1 (E); no longer U203.6 (LED0)
- net at R207.1: now also U203.10 (LED4); no longer U202.6 (J)
- net at R207.2: now also U202.6 (J); no longer U203.10 (LED4)
- net at U203.11 (LED5): now also R208.1; no longer R208.2
- net at U203.12 (LED6): now also R209.1; no longer R209.2
- net at U203.7 (LED1): now also R204.1; no longer R204.2
- net at U203.8 (LED2): now also R205.1; no longer R205.2
- net at U202.2 (M): now also R204.2; no longer R204.1
- net at U202.4 (L): now also R205.2; no longer R205.1
- net at U202.7 (D): now also R208.2; no longer R208.1
- net at U202.8 (DP): now also R209.2; no longer R209.1
Other:
- moved on the sheet: R203, R204, R205, R206, R207, R208, R209
Changed lines of the file:
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@@
     (pin "2")
   )
-  (symbol (lib_id "Device:R") (at 111.76 45.72 270) (unit 1)
+  (symbol (lib_id "Device:R") (at 111.76 45.72 90) (unit 1)
     (in_bom yes) (on_board yes)
     (property "Reference" "R206" (id 0) (at 106.68 44.45 90))
     (property "Value" "330" (id 1) (at 111.76 45.72 90))
-    (property "Footprint" "Resistor_SMD:R_0805_2012Metric" (id 2) (at 111.76 43.942 90)
+    (property "Footprint" "Resistor_SMD:R_0805_2012Metric" (id 2) (at 111.76 47.498 90)
       (effects (font (size 1.27 1.27)) hide)
     )
@@
     (pin "2")
   )
-  (symbol (lib_id "Device:R") (at 111.76 35.56 270) (unit 1)
+  (symbol (lib_id "Device:R") (at 111.76 35.56 90) (unit 1)
     (in_bom yes) (on_board yes)
     (property "Reference" "R203" (id 0) (at 106.68 34.29 90))
     (property "Value" "330" (id 1) (at 111.76 35.56 90))
-    (property "Footprint" "Resistor_SMD:R_0805_2012Metric" (id 2) (at 111.76 33.782 90)
+    (property "Footprint" "Resistor_SMD:R_0805_2012Metric" (id 2) (at 111.76 37.338 90)
       (effects (font (size 1.27 1.27)) hide)
     )
@@
     (pin "2")
   )
-  (symbol (lib_id "Device:R") (at 111.76 48.26 270) (unit 1)
+  (symbol (lib_id "Device:R") (at 111.76 48.26 90) (unit 1)
     (in_bom yes) (on_board yes)
     (property "Reference" "R207" (id 0) (at 106.68 46.99 90))
     (property "Value" "330" (id 1) (at 111.76 48.26 90))
-    (property "Footprint" "Resistor_SMD:R_0805_2012Metric" (id 2) (at 111.76 46.482 90)
+    (property "Footprint" "Resistor_SMD:R_0805_2012Metric" (id 2) (at 111.76 50.038 90)
       (effects (font (size 1.27 1.27)) hide)
     )
@@
     (pin "6")
   )
-  (symbol (lib_id "Device:R") (at 111.76 38.1 270) (unit 1)
+  (symbol (lib_id "Device:R") (at 111.76 38.1 90) (unit 1)
     (in_bom yes) (on_board yes)
     (property "Reference" "R204" (id 0) (at 106.68 36.83 90))
     (property "Value" "330" (id 1) (at 111.76 38.1 90))
-    (property "Footprint" "Resistor_SMD:R_0805_2012Metric" (id 2) (at 111.76 36.322 90)
+    (property "Footprint" "Resistor_SMD:R_0805_2012Metric" (id 2) (at 111.76 39.878 90)
       (effects (font (size 1.27 1.27)) hide)
     )
@@
     (pin "2")
   )
-  (symbol (lib_id "Device:R") (at 111.76 43.18 270) (unit 1)
+  (symbol (lib_id "Device:R") (at 111.76 43.18 90) (unit 1)
     (in_bom yes) (on_board yes)
     (property "Reference" "R205" (id 0) (at 106.68 41.91 90))
     (property "Value" "330" (id 1) (at 111.76 43.18 90))
-    (property "Footprint" "Resistor_SMD:R_0805_2012Metric" (id 2) (at 111.76 41.402 90)
+    (property "Footprint" "Resistor_SMD:R_0805_2012Metric" (id 2) (at 111.76 44.958 90)
       (effects (font (size 1.27 1.27)) hide)
     )
@@
     (pin "2")
   )
-  (symbol (lib_id "Device:R") (at 111.76 53.34 270) (unit 1)
+  (symbol (lib_id "Device:R") (at 111.76 53.34 90) (unit 1)
     (in_bom yes) (on_board yes)
     (property "Reference" "R209" (id 0) (at 106.68 52.07 90))
     (property "Value" "330" (id 1) (at 111.76 53.34 90))
-    (property "Footprint" "Resistor_SMD:R_0805_2012Metric" (id 2) (at 111.76 51.562 90)
+    (property "Footprint" "Resistor_SMD:R_0805_2012Metric" (id 2) (at 111.76 55.118 90)
       (effects (font (size 1.27 1.27)) hide)
     )
@@
     (pin "2")
   )
-  (symbol (lib_id "Device:R") (at 111.76 50.8 270) (unit 1)
+  (symbol (lib_id "Device:R") (at 111.76 50.8 90) (unit 1)
     (in_bom yes) (on_board yes)
     (property "Reference" "R208" (id 0) (at 106.68 49.53 90))
     (property "Value" "330" (id 1) (at 111.76 50.8 90))
-    (property "Footprint" "Resistor_SMD:R_0805_2012Metric" (id 2) (at 111.76 49.022 90)
-      (effects (font (size 1.27 1.27)) hide)
-    )
+    (property "Footprint" "Resistor_SMD:R_0805_2012Metric" (id 2) (at 111.76 52.578 90)
+      (effects (font (size 1.27 1.27)) hide)
+    )

Commit message: replace out of stock components
Parts:
- added C201: 0.1u, Capacitor_SMD:C_0805_2012Metric, symbol Device:C
- added R210: 100k, Resistor_SMD:R_0805_2012Metric, symbol Device:R
- added R219: 6k8, Resistor_SMD:R_0805_2012Metric, symbol Device:R
- U203: value PCA9685PW -> IS32FL3238; symbol Driver_LED:PCA9685PW -> IS32FL3238:IS32FL3238; DK https://www.digikey.no/en/products/detail/PCA9685PW%2c112/5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 -> https://www.digikey.no/en/products/detail/lumissil-microsys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
- renumbered R210 to R211, R211 to R212, R212 to R213, R213 to R214, R214 to R215, R215 to R216, R216 to R217, R217 to R218
Connections:
- net +3V3: now also U201.4 (D2), U201.6 (D1), U203.26 (AD), U203.27 (VCC); no longer U203.1 (A0), U203.28 (VDD), U203.3 (A2), U203.5 (A4)
- net GND: now also U203.15 (GND), U203.28 (GND), C201.2, R210.2, R219.2; no longer U201.2 (S2), U201.5 (S1), U203.2 (A1), U203.24 (A5), U203.25 (EXTCLK), U203.4 (A3)
- net SCL: now also U203.4 (SCL); no longer U203.26 (SCL)
- net SDA: now also U203.3 (SDA); no longer U203.27 (SDA)
- net at R206.1: now also U203.8 (OUT4); no longer U203.9 (LED3)
- net at R203.1: now also U203.5 (OUT1); no longer U203.6 (LED0)
- net at R207.1: now also U203.9 (OUT5); no longer U203.10 (LED4)
- net at R208.1: now also U203.10 (OUT6); no longer U203.11 (LED5)
- net at R209.1: now also U203.11 (OUT7); no longer U203.12 (LED6)
- net at R218.1: now also U203.12 (OUT8); no longer U203.13 (LED7)
- net at R217.1: now also U203.13 (OUT9); no longer U203.15 (LED8)
- net at R204.1: now also U203.6 (OUT2); no longer U203.7 (LED1)
- net at R205.1: now also U203.7 (OUT3); no longer U203.8 (LED2)
- net at U202.11 (C2): now also U201.2 (S2); no longer U201.4 (D2)
- net at U202.16 (C1): now also U201.5 (S1); no longer U201.6 (D1)
- net ~OE: no longer names the net of U203.23 (OUT17)
- new net: R219.1, U203.2 (ISET)
- new net EN: C201.1, R210.1, U203.25 (EN)
- no-connect marks 1 -> 3
Other:
- note added: "I2C address 0b11 = 0x3"
- note removed: "Far away from the PCB"
- note removed: "I2C address 0b1010101=0x55"
- moved on the sheet: R201, R202

Commit message: reroute new components
Parts:
- R219: value 6k8 -> 10k
Connections:
- net +3V3: no longer U203.26 (AD)
- net GND: now also U203.26 (AD)
Other:
- note added: "I2C address 0b00 = 0x0"
- note removed: "I2C address 0b11 = 0x3"
- note removed: "Keep trace physically short for I2C"
Changed lines of the file:
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@@
   (junction (at 162.56 153.67) (diameter 0) (color 0 0 0 0)
   )
-  (junction (at 101.6 121.92) (diameter 0) (color 0 0 0 0)
-  )
   (junction (at 162.56 147.32) (diameter 0) (color 0 0 0 0)
+  )
+  (junction (at 162.56 143.51) (diameter 0) (color 0 0 0 0)
   )
   (junction (at 118.11 153.67) (diameter 0) (color 0 0 0 0)
@@
     (stroke (width 0) (type default) (color 0 0 0 0))
   )
-  (wire (pts (xy 101.6 144.78) (xy 127 144.78))
-    (stroke (width 0) (type default) (color 0 0 0 0))
-  )
   (wire (pts (xy 118.11 50.8) (xy 115.57 50.8))
     (stroke (width 0) (type default) (color 0 0 0 0))
@@
     (stroke (width 0) (type default) (color 0 0 0 0))
   )
-  (wire (pts (xy 127 137.16) (xy 127 144.78))
-    (stroke (width 0) (type default) (color 0 0 0 0))
-  )
   (wire (pts (xy 118.11 45.72) (xy 115.57 45.72))
     (stroke (width 0) (type default) (color 0 0 0 0))
   )
-  (wire (pts (xy 162.56 139.7) (xy 162.56 147.32))
+  (wire (pts (xy 162.56 139.7) (xy 162.56 143.51))
     (stroke (width 0) (type default) (color 0 0 0 0))
   )
@@
     (stroke (width 0) (type default) (color 0 0 0 0))
   )
+  (wire (pts (xy 127 137.16) (xy 127 143.51))
+    (stroke (width 0) (type default) (color 0 0 0 0))
+  )
   (wire (pts (xy 148.59 40.64) (xy 160.02 40.64))
     (stroke (width 0) (type default) (color 0 0 0 0))
@@
     (stroke (width 0) (type default) (color 0 0 0 0))
   )
+  (wire (pts (xy 127 143.51) (xy 162.56 143.51))
+    (stroke (width 0) (type default) (color 0 0 0 0))
+  )
   (wire (pts (xy 138.43 40.64) (xy 140.97 40.64))
     (stroke (width 0) (type default) (color 0 0 0 0))
@@
     (stroke (width 0) (type default) (color 0 0 0 0))
   )
+  (wire (pts (xy 162.56 143.51) (xy 162.56 147.32))
+    (stroke (width 0) (type default) (color 0 0 0 0))
+  )
   (wire (pts (xy 95.25 154.94) (xy 95.25 149.86))
     (stroke (width 0) (type default) (color 0 0 0 0))
@@
     (stroke (width 0) (type default) (color 0 0 0 0))
   )
-  (wire (pts (xy 101.6 121.92) (xy 101.6 144.78))
-    (stroke (width 0) (type default) (color 0 0 0 0))
-  )
   (wire (pts (xy 107.95 99.06) (xy 107.95 106.68))
     (stroke (width 0) (type default) (color 0 0 0 0))
@@
     (stroke (width 0) (type default) (color 0 0 0 0))
   )
-  (text "I2C address\n0b11 = 0x3" (at 127 139.7 0)
-    (effects (font (size 1.27 1.27)) (justify left bottom))
-  )
-  (text "Keep trace physically short for I2C" (at 119.38 160.02 0)
+  (text "I2C address\n0b00 = 0x0" (at 127 139.7 0)
     (effects (font (size 1.27 1.27)) (justify left bottom))
   )
@@
     (in_bom yes) (on_board yes)
     (property "Reference" "R219" (id 0) (at 156.21 137.16 90))
-    (property "Value" "6k8" (id 1) (at 156.21 139.7 90))
+    (property "Value" "10k" (id 1) (at 156.21 139.7 90))
     (property "Footprint" "Resistor_SMD:R_0805_2012Metric" (id 2) (at 156.21 141.478 90)
       (effects (font (size 1.27 1.27)) hide)

Commit message: påske
Parts:
- removed R203, R204, R205, R206, R207, R208, R209, R211, R212, R213, R214, R215, R216, R217, R218: 330, Resistor_SMD:R_0805_2012Metric, symbol Device:R
- removed U202: LTP-3784E, LTP-3784E:LTP-3784E, symbol ltp3784E:LTP-3784E
- added U202: XAMR14A2, LTP-3784E:LTP-3784E, symbol XAMR14A2:XAMR14A2
- U203: value IS32FL3238 -> (none); footprint Package_SO:TSSOP-28_4.4x9.7mm_P0.65mm -> (none); DK https://www.digikey.no/en/products/detail/lumissil-microsys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 -> https://www.digikey.no/no/products/detail/lumissil-microsys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
Connections:
- net at U203.16 (OUT10): now also U202.12 (A)
- net at U203.8 (OUT4): now also U202.5 (L)
- net at U203.20 (OUT14): now also U202.17 (G)
- net at U203.5 (OUT1): now also U202.1 (E)
- net at U203.9 (OUT5): now also U202.6 (K)
- net at U203.21 (OUT15): now also U202.18 (F)
- net at U203.10 (OUT6): now also U202.7 (D)
- net at U203.11 (OUT7): now also U202.8 (DP)
- net at U203.12 (OUT8): now also U202.9 (C)
- net at U203.13 (OUT9): now also U202.10 (B)
- net at U203.17 (OUT11): now also U202.13 (P)
- net at U203.18 (OUT12): now also U202.14 (J)
- net at U203.19 (OUT13): now also U202.15 (H)
- net at U203.6 (OUT2): now also U202.2 (N)
- net at U203.7 (OUT3): now also U202.4 (M)
- net at U201.2 (S2): now also U202.16 (DIG1)
- net at U201.5 (S1): now also U202.11 (DIG2)
Other:
- moved on the sheet: U201

Commit message: final component changes
Parts:
- removed U202: XAMR14A2, LTP-3784E:LTP-3784E, symbol XAMR14A2:XAMR14A2
- added U202: (no value), symbol HDSP-A22C:HDSP-A22C
- C201: value 0.1u -> (none); footprint Capacitor_SMD:C_0805_2012Metric -> (none)
- R201, R202: value 4k7 -> (none); footprint Resistor_SMD:R_0805_2012Metric_Pad1.20x1.40mm_HandSolder -> (none)
- R203: renamed from R210; value 100k -> (none); footprint Resistor_SMD:R_0805_2012Metric -> (none)
- R204: renamed from R219; value 10k -> (none); footprint Resistor_SMD:R_0805_2012Metric -> (none)
- U201: value QS6K1FRATR -> (none); footprint QS6K1FRA:QS6K1FRA -> (none)
Connections:
- net at U201.2 (S2): now also U202.16 (DIG1)
- net at U201.5 (S1): now also U202.11 (DIG2)
- net at U203.5 (OUT1): now also U202.1 (E)
- net at U203.13 (OUT9): now also U202.10 (B)
- net at U203.16 (OUT10): now also U202.12 (A)
- net at U203.17 (OUT11): now also U202.13 (N)
- net at U203.18 (OUT12): now also U202.14 (H)
- net at U203.19 (OUT13): now also U202.15 (G)
- net at U203.20 (OUT14): now also U202.17 (P)
- net at U203.21 (OUT15): now also U202.18 (F)
- net at U203.6 (OUT2): now also U202.2 (M)
- net at U203.7 (OUT3): now also U202.4 (L)
- net at U203.8 (OUT4): now also U202.5 (K)
- net at U203.9 (OUT5): now also U202.6 (J)
- net at U203.10 (OUT6): now also U202.7 (D)
- net at U203.11 (OUT7): now also U202.8 (DP)
- net at U203.12 (OUT8): now also U202.9 (C)
Changed lines of the file:
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@@
     (in_bom yes) (on_board yes)
     (property "Reference" "R202" (id 0) (at 101.6 152.4 90))
-    (property "Value" "4k7" (id 1) (at 101.6 154.94 90))
-    (property "Footprint" "Resistor_SMD:R_0805_2012Metric_Pad1.20x1.40mm_HandSolder" (id 2) (at 101.6 156.718 90)
+    (property "Value" "" (id 1) (at 101.6 154.94 90))
+    (property "Footprint" "" (id 2) (at 101.6 156.718 90)
       (effects (font (size 1.27 1.27)) hide)
     )
@@
       (effects (font (size 1.27 1.27)) (justify left))
     )
-    (property "Value" "QS6K1FRATR" (id 1) (at 138.43 80.01 90)
+    (property "Value" "" (id 1) (at 138.43 80.01 90)
       (effects (font (size 1.27 1.27)) (justify left))
     )
-    (property "Footprint" "QS6K1FRA:QS6K1FRA" (id 2) (at 119.38 76.2 0)
+    (property "Footprint" "" (id 2) (at 119.38 76.2 0)
       (effects (font (size 1.27 1.27)) hide)
     )
@@
   (symbol (lib_id "Device:R") (at 156.21 139.7 90) (unit 1)
     (in_bom yes) (on_board yes)
-    (property "Reference" "R219" (id 0) (at 156.21 137.16 90))
-    (property "Value" "10k" (id 1) (at 156.21 139.7 90))
-    (property "Footprint" "Resistor_SMD:R_0805_2012Metric" (id 2) (at 156.21 141.478 90)
+    (property "Reference" "R204" (id 0) (at 156.21 137.16 90))
+    (property "Value" "" (id 1) (at 156.21 139.7 90))
+    (property "Footprint" "" (id 2) (at 156.21 141.478 90)
       (effects (font (size 1.27 1.27)) hide)
     )
@@
     (pin "2")
   )
-  (symbol (lib_id "Device:R") (at 101.6 149.86 90) (unit 1)
-    (in_bom yes) (on_board yes)
-    (property "Reference" "R201" (id 0) (at 101.6 147.32 90))
-    (property "Value" "4k7" (id 1) (at 101.6 149.86 90))
-    (property "Footprint" "Resistor_SMD:R_0805_2012Metric_Pad1.20x1.40mm_HandSolder" (id 2) (at 101.6 151.638 90)
+  (symbol (lib_id "HDSP-A22C:HDSP-A22C") (at 128.27 44.45 0) (unit 1)
+    (in_bom yes) (on_board yes) (fields_autoplaced)
+    (property "Reference" "U202" (id 0) (at 128.27 29.4472 0))
+    (property "Value" "" (id 1) (at 128.27 31.9841 0))
+    (property "Footprint" "" (id 2) (at 128.27 44.45 0)
       (effects (font (size 1.27 1.27)) hide)
     )
-    (property "Datasheet" "~" (id 3) (at 101.6 149.86 0)
+    (property "Datasheet" "" (id 3) (at 128.27 44.45 0)
       (effects (font (size 1.27 1.27)) hide)
     )
-    (pin "1")
-    (pin "2")
-  )
-  (symbol (lib_id "Device:R") (at 138.43 153.67 90) (unit 1)
-    (in_bom yes) (on_board yes)
-    (property "Reference" "R210" (id 0) (at 138.43 151.13 90))
-    (property "Value" "100k" (id 1) (at 138.43 153.67 90))
-    (property "Footprint" "Resistor_SMD:R_0805_2012Metric" (id 2) (at 138.43 155.448 90)
-      (effects (font (size 1.27 1.27)) hide)
-    )
-    (property "Datasheet" "~" (id 3) (at 138.43 153.67 0)
-      (effects (font (size 1.27 1.27)) hide)
-    )
-    (pin "1")
-    (pin "2")
-  )
-  (symbol (lib_id "XAMR14A2:XAMR14A2") (at 128.27 44.45 0) (unit 1)
-    (in_bom yes) (on_board yes) (fields_autoplaced)
-    (property "Reference" "U202" (id 0) (at 128.27 27.94 0))
-    (property "Value" "XAMR14A2" (id 1) (at 128.27 30.48 0))
-    (property "Footprint" "LTP-3784E:LTP-3784E" (id 2) (at 128.905 48.26 0)
-      (effects (font (size 1.27 1.27)) hide)
-    )
-    (property "Datasheet" "https://www.sunledusa.com/products/spec/XAMR14A2.pdf" (id 3) (at 128.905 48.26 0)
-      (effects (font (size 1.27 1.27)) hide)
-    )
-    (property "DK" "https://www.digikey.no/no/products/detail/sunled/XAMR14A2/4902135" (id 4) (at 128.27 44.45 0)
+    (property "DK" "https://www.digikey.no/no/products/detail/broadcom-limited/HDSP-A22C/3589050" (id 4) (at 128.27 44.45 0)
       (effects (font (size 1.27 1.27)) hide)
     )
@@
     (pin "9")
   )
+  (symbol (lib_id "Device:R") (at 101.6 149.86 90) (unit 1)
+    (in_bom yes) (on_board yes)
+    (property "Reference" "R201" (id 0) (at 101.6 147.32 90))
+    (property "Value" "" (id 1) (at 101.6 149.86 90))
+    (property "Footprint" "" (id 2) (at 101.6 151.638 90)
+      (effects (font (size 1.27 1.27)) hide)
+    )
+    (property "Datasheet" "~" (id 3) (at 101.6 149.86 0)
+      (effects (font (size 1.27 1.27)) hide)
+    )
+    (pin "1")
+    (pin "2")
+  )
+  (symbol (lib_id "Device:R") (at 138.43 153.67 90) (unit 1)
+    (in_bom yes) (on_board yes)
+    (property "Reference" "R203" (id 0) (at 138.43 151.13 90))
+    (property "Value" "" (id 1) (at 138.43 153.67 90))
+    (property "Footprint" "" (id 2) (at 138.43 155.448 90)
+      (effects (font (size 1.27 1.27)) hide)
+    )
+    (property "Datasheet" "~" (id 3) (at 138.43 153.67 0)
+      (effects (font (size 1.27 1.27)) hide)
+    )
+    (pin "1")
+    (pin "2")
+  )
   (symbol (lib_id "power:+3V3") (at 95.25 147.32 0) (unit 1)
     (in_bom yes) (on_board yes)
@@
       (effects (font (size 1.27 1.27)) (justify left))
     )
-    (property "Value" "0.1u" (id 1) (at 144.78 146.05 90)
+    (property "Value" "" (id 1) (at 144.78 146.05 90)
       (effects (font (size 1.27 1.27)) (justify left))
     )
-    (property "Footprint" "Capacitor_SMD:C_0805_2012Metric" (id 2) (at 142.24 146.3548 0)
+    (property "Footprint" "" (id 2) (at 142.24 146.3548 0)
       (effects (font (size 1.27 1.27)) hide)
     )
@@
   )
   (symbol (lib_id "IS32FL3238:IS32FL3238") (at 128.27 121.92 90) (unit 1)
-    (in_bom yes) (on_board yes) (fields_autoplaced)
-    (property "Reference" "U203" (id 0) (at 97.79 118.3386 90))
-    (property "Value" "" (id 1) (at 97.79 120.8786 90))
+    (in_bom yes) (on_board yes)
+    (property "Reference" "U203" (id 0) (at 128.27 119.38 90))
+    (property "Value" "" (id 1) (at 128.27 123.19 90))
     (property "Footprint" "" (id 2) (at 127 121.92 0)
       (effects (font (size 1.27 1.27)) hide)
